File: MPPT Eval Board/MPPT.kicad_sch (KiCad schematic)
At the start: 16 parts, among them Q4 UMWIRLML6344TR, Q5 UMWIRLML6344TR, U4 LTC4162EUFD-LAD-TRPBF

Commit message: Added I2C pullups and board ready for layout
Parts:
- removed C6: 100n, Capacitor_SMD:C_0603_1608Metric, symbol Device:C_Small
- added C46, C49: 10u, Capacitor_SMD:C_1210_3225Metric, symbol Device:C_Small
- added R68, R71: 0R, Resistor_SMD:R_0603_1608Metric, symbol Device:R_Small
- added TP19, TP22: TestPoint, Connector_Pin:Pin_D1.0mm_L10.0mm, symbol Connector:TestPoint
Connections:
- net GND: now also C46.1, C49.2, R68.1, R71.1; no longer U4.13 (SCL), U4.14 (SDA)
- net VIN: now also Q4.2 (S); no longer Q4.3 (D)
- net VOUT: now also C49.1
- net at Q5.3 (D), R1.2, U4.27 (VOUT)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: now also C46.2
- net at R1.1, U4.5 (CLP): now also Q4.3 (D); no longer Q4.2 (S)
- net INFET: now reaches Q4.1 (G), U4.6 (INFET)
- new net: R68.2, TP22.1, U4.13 (SCL)
- new net: R71.2, TP19.1, U4.14 (SDA)
Other:
- moved on the sheet: TP16
