File: MPPT Eval Board/battery.kicad_sch (KiCad schematic)
At the start: 9 parts, among them J3 Keystone-1042, J4 Keystone-1042

Commit message: Initial layout: need to thicken power traces and make inductor loop tighter
Parts:
- J3, J4: footprint Argus-Misc:Keystone_1042 -> Argus-Miscellaneous:Keystone_1042
Changed lines of the file:
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@@
 			)
 		)
-		(property "Footprint" "Argus-Misc:Keystone_1042"
+		(property "Footprint" "Argus-Miscellaneous:Keystone_1042"
 			(at 105.41 78.74 0)
 			(hide yes)
@@
 			)
 		)
-		(property "Footprint" "Argus-Misc:Keystone_1042"
+		(property "Footprint" "Argus-Miscellaneous:Keystone_1042"
 			(at 133.35 78.74 0)
 			(hide yes)
