File: MPPT Eval Board/MPPT Eval Board.kicad_pcb (KiCad board)
At the start: 2 copper layers, 390 x 205 mm, 303 parts, among them J3 Keystone-1042, J4 Keystone-1042, J5 Keystone-1042, J6 Keystone-1042, Q1 SIRA99DP-T1-GE3, Q10 UMWIRLML6344TR, Q11 SIRA99DP-T1-GE3, Q12 SIRA99DP-T1-GE3, Q4 UMWIRLML6344TR, Q5 UMWIRLML6344TR, Q6 UMWIRLML6344TR, Q7 UMWIRLML6344TR, Q9 UMWIRLML6344TR, U1 LTC4412xS6, U10 LTC3130IUDC, U11 LTC3130IUDC, U12 LTC3130IUDC, U4 LTC4162EUFD-LAD-TRPBF, U5 LTC4162EUFD-LAD-TRPBF, U7 LTC4162EUFD-LAD-TRPBF, U8 LTC4412xS6, U9 LTC4412xS6

Commit message: Applying changes to MPPC implementation
Routing:
- net GND: track 366.6 -> 309.0 mm, vias 56 -> 61
- net /MPPC Implementation/VSOLAR1: track 455.7 -> 461.5 mm
- net /MPPC Implementation/VCHRG: track 388.8 -> 389.9 mm
- net Net-(Q7-S): track 14.5 -> 15.3 mm
- net /MPPC Implementation/MPPC1/VCC: track 40.2 -> 39.6 mm

Commit message: READY FOR FINAL LAYOUT REVIEW
Parts:
- moved Q7 11.9 mm to (200.4, 263.1), turned to 90 degrees
- moved Q10 11.6 mm to (200.0, 368.0), turned to 90 degrees
- moved L1 11.5 mm to (290.5, 263.5), turned to 90 degrees
- moved L2 11.5 mm to (194.5, 263.5), turned to 90 degrees
- moved Q5 11.5 mm to (296.0, 263.0), turned to 90 degrees
- moved L3 11.4 mm to (194.5, 368.0), turned to 90 degrees
- moved C48 5.51 mm to (189.0, 366.0), turned to -90 degrees
- moved C46 5.39 mm to (285.0, 261.5), turned to -90 degrees
- moved C47 5.39 mm to (189.0, 261.5), turned to -90 degrees
- moved C7 3.65 mm to (283.5, 266.0)
- moved C11 3.54 mm to (187.8, 266.0)
- moved C16 2.42 mm to (188.0, 369.5)
Routing:
- net /MPPT Implementation/VCHRG: track 538.1 -> 590.7 mm
- net Net-(Q10-S): track 14.5 -> 36.8 mm
- net Net-(Q7-S): track 15.3 -> 36.5 mm
- net /MPPT Implementation/VSOLAR1: track 357.6 -> 377.3 mm
- net Net-(Q7-G): track 2.88 -> 21.8 mm
- net Net-(Q5-S): track 14.5 -> 32.9 mm
- net GND: track 309.0 -> 292.0 mm
- net Net-(Q10-G): track 2.88 -> 18.9 mm
- net Net-(Q5-G): track 2.88 -> 18.7 mm
- net Net-(Q7-D): track 24.8 -> 34.7 mm
- net Net-(Q5-D): track 24.8 -> 33.7 mm
- net Net-(Q10-D): track 24.8 -> 33.1 mm
- net /MPPC Implementation/VCHRG: track 389.9 -> 395.6 mm
- net Net-(C11-Pad2): track 13.1 -> 16.4 mm
- net Net-(C7-Pad2): track 13.1 -> 16.3 mm
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